File: Data_Logger_KiCAD/IMU.kicad_sch (KiCad schematic)
At the start: 0 parts

Commit message: Organization and LSM6DSO32 (IMU) schematic
Parts:
- added C1, C2: 100 nF, symbol Device:C
- added U1: LSM6DSO32TR, LSM6DSO32TR:XDCR_LSM6DSO32TR, symbol LSM6DSO32:LSM6DSO32TR
Connections:
- new net: C2.1, U1.8 (VDD)
- new net: C1.1, U1.5 (VDDIO)
- new net: U1.10 (NC), U1.11 (NC)
- new net CS_IMU: U1.12 (CS)
- new net GND: C1.2, C2.2, U1.2 (SDX), U1.3 (SCX), U1.6 (GND), U1.7 (GND)
- new net SDI: U1.14 (SDA)
- new net SDO: U1.1 (SDO/SA0)
- new net SPC: U1.13 (SCL)
- no-connect marks 0 -> 2
Other:
- note added: "May need to connect interupts (INT1 and INT2). Double check."

Commit message: add footprint/LCSC to parts
Parts:
- removed C1, C2: 100 nF, symbol Device:C
- removed U1: LSM6DSO32TR, LSM6DSO32TR:XDCR_LSM6DSO32TR, symbol LSM6DSO32:LSM6DSO32TR
Connections:
- no-connect marks 2 -> 0
Other:
- note removed: "May need to connect interupts (INT1 and INT2). Double check."
