File: Data_Logger_KiCAD/IMU.kicad_sch (KiCad schematic)
At the start: 9 parts, among them U1 LSM6DSO32TR, U3 ADXL375, U5 BMI088

Commit message: layout power plane
Connections:
- net IMU_CS renamed ~{IMU_CS}
Changed lines of the file:
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@@
 		)
 	)
-	(hierarchical_label "IMU_CS"
+	(hierarchical_label "~{IMU_CS}"
 		(shape input)
 		(at 88.9 59.69 0)

Commit message: remove units for extraction
Parts:
- C16, C17: value 100 nF -> 100n
Changed lines of the file:
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@@
 			)
 		)
-		(property "Value" "100 nF"
+		(property "Value" "100n"
 			(at 134.62 54.6099 0)
 			(effects
@@
 			)
 		)
-		(property "Value" "100 nF"
+		(property "Value" "100n"
 			(at 120.65 54.6099 0)
 			(effects
