File: Data_Logger_KiCAD/GPS.kicad_sch (KiCad schematic)
At the start: 0 parts

Commit message: Radio Layout V1.0
Parts:
- added C1: 1u, Capacitor_SMD:C_0402_1005Metric, symbol Device:C
- added C2: 100n, Capacitor_SMD:C_0402_1005Metric, symbol Device:C
- added U1: MAX-M10S, RF_GPS:ublox_MAX, symbol RF_GPS:MAX-M10S
Connections:
- new net +3.3V: C1.1, C2.1, U1.7 (VCC_IO), U1.8 (VCC)
- new net Antenna: U1.11 (RF_IN)
- new net EXTINT: U1.5 (EXTINT)
- new net GND: C1.2, C2.2, U1.1 (GND), U1.10 (GND), U1.12 (GND)
- new net SCL: U1.17 (SCL)
- new net SDA: U1.16 (SDA)
- no-connect marks 0 -> 9
Other:
- note added: "1 - GND 2 - open (UART) 3 - open (UART) 4 - open (timepulse not needed) 5 - EXTINT (used for sleep awakening) 6 - open (no backup supply) 7 - 3.3V (I2C logic level) 8 - 3.3V in (need cap) 9 - open (reset not needed) 10 - GND (combined with 1) 11 - patch antenna connection 12 - GND (combined with 1) 13 - open (to ext LNA output) 14 - open (no active antenna) 15 - open (3.3V mode) 16 - I2C data 17 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"
- note added: "I/O table"

Commit message: minor updates
Parts:
- added AE1: Antenna, symbol Device:Antenna
- added D2: LED, LED_SMD:LED_0603_1608Metric, symbol Device:LED
- added R25: 49.9, Resistor_SMD:R_0402_1005Metric, symbol Device:R_Small
Connections:
- net TIMEPULSE: now reaches U1.4 (TIMEPULSE)
- net TIMEPULSE: now also D2.1 (K)
- net Antenna: no longer names the net of U1.11 (RF_IN)
- net Antenna: now also AE1.1 (A)
- new net: D2.2 (A), R25.1
- new net +3V3: R25.2
- no-connect marks 9 -> 8

Commit message: Aggregated sub schematics into single primary schematic
Parts:
- U4: renamed from U1; footprint RF_GPS:ublox_MAX -> Package_LGA:LGA-8_3x5mm_P1.25mm
- renumbered AE1 to AE2, C1 to C29, C2 to C30, R25 to R10
Changed lines of the file:
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@@
 		(dnp no)
 		(fields_autoplaced yes)
-		(property "Reference" "R25"
+		(property "Reference" "R10"
 			(at 152.4 78.74 90)
 			(effects
@@
 		(instances
 			(project "Data_Logger_Board"
-				(path "/db968e42-3ace-4cc9-9096-9d8f48135c40/caa54f87-1e96-4d4c-b6a8-b81d14fe08af"
-					(reference "R25")
+				(path "/db968e42-3ace-4cc9-9096-9d8f48135c40/795ab2be-9db7-4254-b05c-ac2b60177344/bd56c2d0-6430-41ab-a92d-256e41365a97"
+					(reference "R10")
 					(unit 1)
 				)
@@
 		(dnp no)
 		(fields_autoplaced yes)
-		(property "Reference" "C2"
+		(property "Reference" "C30"
 			(at 109.22 46.9899 0)
 			(effects
@@
 		(instances
 			(project "Data_Logger_Board"
-				(path "/db968e42-3ace-4cc9-9096-9d8f48135c40/caa54f87-1e96-4d4c-b6a8-b81d14fe08af"
-					(reference "C2")
+				(path "/db968e42-3ace-4cc9-9096-9d8f48135c40/795ab2be-9db7-4254-b05c-ac2b60177344/bd56c2d0-6430-41ab-a92d-256e41365a97"
+					(reference "C30")
 					(unit 1)
 				)
@@
 		(on_board yes)
 		(dnp no)
-		(property "Reference" "C1"
+		(property "Reference" "C29"
 			(at 99.06 46.9899 0)
 			(effects
@@
 		(instances
 			(project "Data_Logger_Board"
-				(path "/db968e42-3ace-4cc9-9096-9d8f48135c40/caa54f87-1e96-4d4c-b6a8-b81d14fe08af"
-					(reference "C1")
+				(path "/db968e42-3ace-4cc9-9096-9d8f48135c40/795ab2be-9db7-4254-b05c-ac2b60177344/bd56c2d0-6430-41ab-a92d-256e41365a97"
+					(reference "C29")
 					(unit 1)
 				)
@@
 		(dnp no)
 		(fields_autoplaced yes)
-		(property "Reference" "#PWR068"
+		(property "Reference" "#PWR053"
 			(at 157.48 86.36 0)
 			(effects
@@
 		(instances
 			(project "Data_Logger_Board"
-				(path "/db968e42-3ace-4cc9-9096-9d8f48135c40/caa54f87-1e96-4d4c-b6a8-b81d14fe08af"
-					(reference "#PWR068")
+				(path "/db968e42-3ace-4cc9-9096-9d8f48135c40/795ab2be-9db7-4254-b05c-ac2b60177344/bd56c2d0-6430-41ab-a92d-256e41365a97"
+					(reference "#PWR053")
 					(unit 1)
 				)
@@
 		(dnp no)
 		(fields_autoplaced yes)
-		(property "Reference" "#PWR01"
+		(property "Reference" "#PWR054"
 			(at 121.92 102.87 0)
 			(effects
@@
 		(instances
 			(project "Data_Logger_Board"
-				(path "/db968e42-3ace-4cc9-9096-9d8f48135c40/caa54f87-1e96-4d4c-b6a8-b81d14fe08af"
-					(reference "#PWR01")
+				(path "/db968e42-3ace-4cc9-9096-9d8f48135c40/795ab2be-9db7-4254-b05c-ac2b60177344/bd56c2d0-6430-41ab-a92d-256e41365a97"
+					(reference "#PWR054")
 					(unit 1)
 				)
@@
 		(dnp no)
 		(fields_autoplaced yes)
-		(property "Reference" "#PWR04"
+		(property "Reference" "#PWR052"
 			(at 105.41 60.96 0)
 			(effects
@@
 		(instances
 			(project "Data_Logger_Board"
-				(path "/db968e42-3ace-4cc9-9096-9d8f48135c40/caa54f87-1e96-4d4c-b6a8-b81d14fe08af"
-					(reference "#PWR04")
+				(path "/db968e42-3ace-4cc9-9096-9d8f48135c40/795ab2be-9db7-4254-b05c-ac2b60177344/bd56c2d0-6430-41ab-a92d-256e41365a97"
+					(reference "#PWR052")
 					(unit 1)
 				)
@@
 		(dnp no)
 		(fields_autoplaced yes)
-		(property "Reference" "AE1"
+		(property "Reference" "AE2"
 			(at 148.59 64.1349 0)
 			(effects
@@
 		)
 		(instances
-			(project ""
-				(path "/db968e42-3ace-4cc9-9096-9d8f48135c40/caa54f87-1e96-4d4c-b6a8-b81d14fe08af"
-					(reference "AE1")
+			(project "Data_Logger_Board"
+				(path "/db968e42-3ace-4cc9-9096-9d8f48135c40/795ab2be-9db7-4254-b05c-ac2b60177344/bd56c2d0-6430-41ab-a92d-256e41365a97"
+					(reference "AE2")
 					(unit 1)
 				)
@@
 		(dnp no)
 		(fields_autoplaced yes)
-		(property "Reference" "#PWR02"
+		(property "Reference" "#PWR050"
 			(at 116.84 45.72 0)
 			(effects
@@
 		(instances
 			(project "Data_Logger_Board"
-				(path "/db968e42-3ace-4cc9-9096-9d8f48135c40/caa54f87-1e96-4d4c-b6a8-b81d14fe08af"
-					(reference "#PWR02")
+				(path "/db968e42-3ace-4cc9-9096-9d8f48135c40/795ab2be-9db7-4254-b05c-ac2b60177344/bd56c2d0-6430-41ab-a92d-256e41365a97"
+					(reference "#PWR050")
 					(unit 1)
 				)
@@
 		(dnp no)
 		(fields_autoplaced yes)
-		(property "Reference" "#PWR03"
+		(property "Reference" "#PWR051"
 			(at 95.25 60.96 0)
 			(effects
@@
 		(instances
 			(project "Data_Logger_Board"
-				(path "/db968e42-3ace-4cc9-9096-9d8f48135c40/caa54f87-1e96-4d4c-b6a8-b81d14fe08af"
-					(reference "#PWR03")
+				(path "/db968e42-3ace-4cc9-9096-9d8f48135c40/795ab2be-9db7-4254-b05c-ac2b60177344/bd56c2d0-6430-41ab-a92d-256e41365a97"
+					(reference "#PWR051")
 					(unit 1)
 				)
@@
 		(dnp no)
 		(fields_autoplaced yes)
-		(property "Reference" "U1"
+		(property "Reference" "U4"
 			(at 124.0633 93.98 0)
 			(effects
@@
 			)
 		)
-		(property "Footprint" "RF_GPS:ublox_MAX"
+		(property "Footprint" "Package_LGA:LGA-8_3x5mm_P1.25mm"
 			(at 132.08 92.71 0)
 			(effects
@@
 		(instances
 			(project "Data_Logger_Board"
-				(path "/db968e42-3ace-4cc9-9096-9d8f48135c40/caa54f87-1e96-4d4c-b6a8-b81d14fe08af"
-					(reference "U1")
+				(path "/db968e42-3ace-4cc9-9096-9d8f48135c40/795ab2be-9db7-4254-b05c-ac2b60177344/bd56c2d0-6430-41ab-a92d-256e41365a97"
+					(reference "U4")
 					(unit 1)
 				)
@@
 		(instances
 			(project "Data_Logger_Board"
-				(path "/db968e42-3ace-4cc9-9096-9d8f48135c40/caa54f87-1e96-4d4c-b6a8-b81d14fe08af"
+				(path "/db968e42-3ace-4cc9-9096-9d8f48135c40/795ab2be-9db7-4254-b05c-ac2b60177344/bd56c2d0-6430-41ab-a92d-256e41365a97"
 					(reference "D2")
 					(unit 1)

Commit message: add footprint/LCSC to parts
Parts:
- C29: LCSC (none) -> C52923
- C30: LCSC (none) -> C1525
Changed lines of the file:
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@@
+			)
+		)
+		(property "LCSC" "C1525"
+			(at 105.41 48.26 0)
+			(effects
+				(font
+					(size 1.27 1.27)
+				)
+				(hide yes)
 			)
 		)
@@
 			(at 95.25 48.26 0)
 			(effects
+				(font
+					(size 1.27 1.27)
+				)
+				(hide yes)
+			)
+		)
+		(property "LCSC" "C52923"
+			(at 95.25 48.26 0)
+			(effects

Commit message: adding labels and updating IMU sch
Other:
- moved on the sheet: AE2
Changed lines of the file:
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@@
 	(wire
 		(pts
-			(xy 146.05 76.2) (xy 146.05 69.85)
+			(xy 151.13 76.2) (xy 151.13 69.85)
 		)
 		(stroke
@@
 	(wire
 		(pts
-			(xy 137.16 76.2) (xy 146.05 76.2)
+			(xy 137.16 76.2) (xy 151.13 76.2)
 		)
 		(stroke
@@
 				)
 				(justify left)
-				(hide yes)
 			)
 		)
@@
 	(symbol
 		(lib_id "Device:Antenna")
-		(at 146.05 64.77 0)
+		(at 151.13 64.77 0)
 		(unit 1)
 		(exclude_from_sim no)
@@
 		(fields_autoplaced yes)
 		(property "Reference" "AE2"
-			(at 148.59 64.1349 0)
+			(at 153.67 64.1349 0)
 			(effects
 				(font
@@
 		)
 		(property "Value" "Antenna"
-			(at 148.59 66.6749 0)
+			(at 153.67 66.6749 0)
 			(effects
 				(font
@@
 		)
 		(property "Footprint" ""
-			(at 146.05 64.77 0)
+			(at 151.13 64.77 0)
 			(effects
 				(font
@@
 		)
 		(property "Datasheet" "~"
-			(at 146.05 64.77 0)
+			(at 151.13 64.77 0)
 			(effects
 				(font
@@
 		)
 		(property "Description" "Antenna"
-			(at 146.05 64.77 0)
-			(effects
-				(font
+			(at 151.13 64.77 0)
+			(effects
+				(font

Commit message: synced sheet pins in Data_Logger_Board_pro
Parts:
- U4: footprint Package_LGA:LGA-8_3x5mm_P1.25mm -> RF_GPS:ublox_MAX
Changed lines of the file:
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@@
 			)
 		)
-		(property "Footprint" "Package_LGA:LGA-8_3x5mm_P1.25mm"
+		(property "Footprint" "RF_GPS:ublox_MAX"
 			(at 132.08 92.71 0)
 			(effects
