File: Data_Logger_KiCAD/MAGNETOMETER.kicad_sch (KiCad schematic)
At the start: 3 parts, among them U11 MMC5983MA

Commit message: fix footprint errors
Parts:
- U11: footprint footprints:MMC5983MA_MEM -> custom:MMC5983MA_MEM
Changed lines of the file:
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@@
 			)
 		)
-		(property "Footprint" "footprints:MMC5983MA_MEM"
+		(property "Footprint" "custom:MMC5983MA_MEM"
 			(at 100.33 62.23 0)
 			(effects

Commit message: footprint + sd tweaks
Parts:
- U11: footprint custom:MMC5983MA_MEM -> Package_LGA:LGA-16_3x3mm_P0.5mm_LayoutBorder3x5y
Changed lines of the file:
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@@
 			)
 		)
-		(property "Footprint" "custom:MMC5983MA_MEM"
+		(property "Footprint" "Package_LGA:LGA-16_3x3mm_P0.5mm_LayoutBorder3x5y"
 			(at 100.33 62.23 0)
 			(effects
