File: Data_Logger_KiCAD/PWR.kicad_sch (KiCad schematic)
At the start: 0 parts

Commit message: added pwr schematic.
Parts:
- added C37: 10u, Capacitor_SMD:C_0603_1608Metric, symbol Device:C
- added Cee: 22u, Capacitor_SMD:C_0603_1608Metric, symbol Device:C
- added U12: AMS1117-3.3, Package_TO_SOT_SMD:SOT-223-3_TabPin2, symbol Regulator_Linear:AMS1117-3.3
Connections:
- new net GND: C37.2, Cee.2, U12.1 (GND)
- new net PWR_IN: C37.1, U12.3 (VI)
- new net PWR_OUT: Cee.1, U12.2 (VO)
