File: Data_Logger_KiCAD/PWR.kicad_sch (KiCad schematic)
At the start: 3 parts, among them U12 AMS1117-3.3

Commit message: rem old files and add LCSC #'s
Parts:
- U12: LCSC (none) -> C6186
Changed lines of the file:
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@@
+			)
+		)
+		(property "LCSC" "C6186"
+			(at 116.84 93.98 0)
+			(effects
+				(font
+					(size 1.27 1.27)
+				)
+				(hide yes)
 			)
 		)

Commit message: update pcb and create .bkp backup
Parts:
- renumbered Cee to C99
Changed lines of the file:
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@@
 		(dnp no)
 		(fields_autoplaced yes)
-		(property "Reference" "Cee"
+		(property "Reference" "C99"
 			(at 138.43 96.5199 0)
 			(effects
@@
 			(project ""
 				(path "/db968e42-3ace-4cc9-9096-9d8f48135c40/795ab2be-9db7-4254-b05c-ac2b60177344/90b9ee1f-09cc-4b5a-82ab-b7ba82166c76"
-					(reference "Cee")
+					(reference "C99")
 					(unit 1)
 				)
