File: Barometers/Barometers.kicad_sch (KiCad schematic)
At the start: 7 parts, among them U1 BMP390L, U3 MS560702BA03-50

Commit message: added footprints to barometer project
Parts:
- C1, C2, C4, C5: footprint (none) -> Capacitor_SMD:C_0402_1005Metric
- R1: footprint (none) -> Resistor_SMD:R_0402_1005Metric
- U1: footprint BMP390L:XDCR_BMP390L -> BMP390:XDCR_BMP390L
- U3: footprint MS56:SON8_MS5611_TEC -> LSM6DSO32:XDCR_LSM6DSO32TR
Changed lines of the file:
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@@
 			)
 		)
-		(property "Footprint" ""
+		(property "Footprint" "Capacitor_SMD:C_0402_1005Metric"
 			(at 120.3452 59.69 0)
 			(effects
@@
 			)
 		)
-		(property "Footprint" ""
+		(property "Footprint" "Resistor_SMD:R_0402_1005Metric"
 			(at 85.09 42.418 90)
 			(effects
@@
 			)
 		)
-		(property "Footprint" "MS56:SON8_MS5611_TEC"
+		(property "Footprint" "LSM6DSO32:XDCR_LSM6DSO32TR"
 			(at 64.77 55.88 0)
 			(effects
@@
 			)
 		)
-		(property "Datasheet" ""
+		(property "Datasheet" "https://www.te.com/usa-en/product-MS560702BA03-50.datasheet.pdf"
 			(at 64.77 55.88 0)
 			(effects
@@
 			)
 		)
-		(property "Footprint" ""
+		(property "Footprint" "Capacitor_SMD:C_0402_1005Metric"
 			(at 103.8352 59.69 0)
 			(effects
@@
 			)
 		)
-		(property "Datasheet" "~"
+		(property "Datasheet" ""
 			(at 102.87 55.88 0)
 			(effects
@@
 			)
 		)
-		(property "Footprint" ""
+		(property "Footprint" "Capacitor_SMD:C_0402_1005Metric"
 			(at 102.5652 134.62 0)
 			(effects
@@
 			)
 		)
-		(property "Footprint" "BMP390L:XDCR_BMP390L"
-			(at 60.96 130.81 0)
-			(effects
-				(font
-					(size 1.27 1.27)
-				)
-				(justify bottom)
-				(hide yes)
-			)
-		)
-		(property "Datasheet" ""
+		(property "Footprint" "BMP390:XDCR_BMP390L"
+			(at 60.96 130.81 0)
+			(effects
+				(font
+					(size 1.27 1.27)
+				)
+				(justify bottom)
+				(hide yes)
+			)
+		)
+		(property "Datasheet" "https://www.bosch-sensortec.com/media/boschsensortec/downloads/datasheets/bst-bmp390-ds002.pdf"
 			(at 60.96 130.81 0)
 			(effects
@@
 			)
 		)
-		(property "Footprint" ""
+		(property "Footprint" "Capacitor_SMD:C_0402_1005Metric"
 			(at 120.3452 134.62 0)
 			(effects
